Commit message: update

File: panda_hand_backup.urdf (robot description, URDF)
Before this commit: robot panda, 10 links, 8 joints
Links:
- removed link ${arm_id}_link8
- added link panda_hand; collision mesh filename=package://franka_description/meshes/collision/hand.stl; visual mesh filename=package://franka_description/meshes/visual/hand.dae
- added link panda_hand_sc; collision cylinder length=0.1 radius=0.05; collision cylinder length=0.1 radius=0.07
- added link panda_hand_tcp
- added link panda_leftfinger; collision box size=17.5e-3 15.2e-3 18.5e-3; collision box size=17.5e-3 7e-3 23.5e-3
- added link panda_rightfinger; collision box size=17.5e-3 15.2e-3 18.5e-3; collision box size=17.5e-3 7e-3 23.5e-3
Joints:
- removed joint ${arm_id}_joint8
- added joint panda_finger_joint1: type prismatic, parent panda_hand, child panda_leftfinger, origin xyz=0 0 0.0584 rpy=0 0 0, axis 0 1 0, limit lower=0.0 upper=0.04 effort=100 velocity=0.2
- added joint panda_finger_joint2: type prismatic, parent panda_hand, child panda_rightfinger, origin xyz=0 0 0.0584 rpy=0 0 0, axis 0 -1 0, limit lower=0.0 upper=0.04 effort=100 velocity=0.2, mimic joint=panda_finger_joint1
- added joint panda_hand_joint: type fixed, parent panda_link8, child panda_hand, origin xyz=0 0 0 rpy=0 0 -0.7853981633974483
- added joint panda_hand_sc_joint: type fixed, parent panda_hand, child panda_hand_sc, origin rpy=0 0 0
- added joint panda_hand_tcp_joint: type fixed, parent panda_hand, child panda_hand_tcp, origin xyz=0 0 0.1034 rpy=0 0 0
